File: Breadboard_Power_Supply.sch (KiCad schematic (older format))
At the start: 20 parts, among them J1 9V Battery, J2 USB_B, J3 Barrel_Jack_Switch, J4 1, J5 2, J6 3, SW1 SW_DIP_x03, U1 AMS1117-5.0, U2 AMS1117-3.3

Commit message: Changed most footprints to SMD + Variable voltage
Parts:
- removed D1: 1N4007, Diode_THT:D_DO-41_SOD81_P7.62mm_Horizontal, symbol Diode:1N4007
- removed J6: 3, Connector_PinHeader_2.54mm:PinHeader_2x03_P2.54mm_Vertical, symbol Connector_Generic:Conn_02x03_Odd_Even
- removed SW1: SW_DIP_x03, Button_Switch_THT:SW_DIP_SPSTx03_Slide_9.78x9.8mm_W7.62mm_P2.54mm, symbol Switch:SW_DIP_x03
- added C1: 0.1uF, Capacitor_SMD:C_1206_3216Metric_Pad1.42x1.75mm_HandSolder, symbol Device:CP_Small
- added C2: 1uF, Capacitor_SMD:C_1206_3216Metric_Pad1.42x1.75mm_HandSolder, symbol Device:CP_Small
- added D1: 1N4148WT, Diode_SMD:D_SOD-523, symbol Diode:1N4148WT
- added DS3: LED, LED_SMD:LED_1206_3216Metric_Pad1.42x1.75mm_HandSolder, symbol Device:LED
- added J6: Conn_02x04_Odd_Even, Connector_PinHeader_2.54mm:PinHeader_2x04_P2.54mm_Vertical_SMD, symbol Connector_Generic:Conn_02x04_Odd_Even
- added R1: 5k, Potentiometer_SMD:Potentiometer_Bourns_3314G_Vertical, symbol Device:R_Variable
- added R2: 240R, Resistor_SMD:R_0805_2012Metric_Pad1.15x1.40mm_HandSolder, symbol Device:R
- added R5: 820R, Resistor_SMD:R_0805_2012Metric_Pad1.15x1.40mm_HandSolder, symbol Device:R
- added SW1: SW_DIP_x04, Button_Switch_SMD:SW_DIP_SPSTx04_Slide_9.78x12.34mm_W8.61mm_P2.54mm, symbol Switch:SW_DIP_x04
- added TP5: TestPoint, TestPoint:TestPoint_Pad_1.0x1.0mm, symbol Connector:TestPoint
- added U1: LM317_3PinPackage, Package_TO_SOT_SMD:SOT-223, symbol Regulator_Linear:LM317_3PinPackage
- C3: renamed from C1; footprint Capacitor_THT:C_Radial_D6.3mm_H11.0mm_P2.50mm -> Capacitor_SMD:C_1206_3216Metric_Pad1.42x1.75mm_HandSolder
- C4: renamed from C2; footprint Capacitor_THT:C_Radial_D6.3mm_H11.0mm_P2.50mm -> Capacitor_SMD:C_1206_3216Metric_Pad1.42x1.75mm_HandSolder
- DS1, DS2: footprint LED_THT:LED_D3.0mm -> LED_SMD:LED_1206_3216Metric_Pad1.42x1.75mm_HandSolder
- J1: footprint Connector_PinHeader_2.54mm:PinHeader_1x02_P2.54mm_Vertical -> Connector_PinHeader_2.54mm:PinHeader_1x02_P2.54mm_Vertical_SMD_Pin1Left
- R3: renamed from R1; footprint Resistor_THT:R_Axial_DIN0207_L6.3mm_D2.5mm_P7.62mm_Horizontal -> Resistor_SMD:R_0805_2012Metric_Pad1.15x1.40mm_HandSolder
- R4: renamed from R2; footprint Resistor_THT:R_Axial_DIN0207_L6.3mm_D2.5mm_P7.62mm_Horizontal -> Resistor_SMD:R_0805_2012Metric_Pad1.15x1.40mm_HandSolder
- renumbered J3 to J2, J2 to J3, U1 to U2, U2 to U3
Connections:
- net +3V3: now also J6.3 (Pin_3), J6.4 (Pin_4), SW1.6
- net +5V: now also J6.1 (Pin_1), J6.2 (Pin_2), SW1.8
- net 3.3V_OUT: now also SW1.3
- net 5V_OUT: now also SW1.1
- net GND: now also J3.4 (GND), C1.2, C2.2, DS3.1 (K), J6.7 (Pin_7), J6.8 (Pin_8), R1.2
- net VDC: now also D1.1 (K), SW1.2
- net VIN: now also C1.1, SW1.7, U1.3 (VI)
- net at J1.2 (Pin_2): now also D1.2 (A)
- new net: R1.1, R2.2, U1.1 (ADJ)
- new net: DS3.2 (A), R5.2
- new net VAR_VLG: J6.5 (Pin_5), J6.6 (Pin_6), R5.1, SW1.5, TP5.1
- new net VAR_VLG_OUT: C2.1, R2.1, SW1.4, U1.2 (VO)
- no-connect marks 3 -> 2
Other:
- note added: "Variable power supply\n"

Commit message: Protection diode changed + Datasheets
Parts:
- D1: value 1N4148WT -> SS22T3G; footprint Diode_SMD:D_SOD-523 -> Diode_SMD:D_SMB
- R4: value 1.5k -> 1k
Other:
- note added: "RED"
- note added: "Use 2k pot\nif available"
Changed lines of the file:
@@
 L Device:LED DS2
 U 1 1 5F8D64C8
-P 4075 4375
-F 0 "DS2" V 4113 4258 50  0000 R CNN
-F 1 "LED" V 4022 4258 50  0000 R CNN
-F 2 "LED_SMD:LED_1206_3216Metric_Pad1.42x1.75mm_HandSolder" H 4075 4375 50  0001 C CNN
-F 3 "~" H 4075 4375 50  0001 C CNN
-	1    4075 4375
+P 4225 4375
+F 0 "DS2" V 4263 4258 50  0000 R CNN
+F 1 "LED" V 4172 4258 50  0000 R CNN
+F 2 "LED_SMD:LED_1206_3216Metric_Pad1.42x1.75mm_HandSolder" H 4225 4375 50  0001 C CNN
+F 3 "~" H 4225 4375 50  0001 C CNN
+	1    4225 4375
 	0    -1   -1   0
 $EndComp
@@
 L Device:R R4
 U 1 1 5F8D64CE
-P 4075 3925
-F 0 "R4" H 4145 3971 50  0000 L CNN
-F 1 "1.5k" H 4145 3880 50  0000 L CNN
-F 2 "Resistor_SMD:R_0805_2012Metric_Pad1.15x1.40mm_HandSolder" V 4005 3925 50  0001 C CNN
-F 3 "~" H 4075 3925 50  0001 C CNN
-	1    4075 3925
+P 4225 3925
+F 0 "R4" H 4295 3971 50  0000 L CNN
+F 1 "1k" H 4295 3880 50  0000 L CNN
+F 2 "Resistor_SMD:R_0805_2012Metric_Pad1.15x1.40mm_HandSolder" V 4155 3925 50  0001 C CNN
+F 3 "~" H 4225 3925 50  0001 C CNN
+	1    4225 3925
 	1    0    0    -1
 $EndComp
@@
 L power:GND #PWR012
 U 1 1 5F8D64DA
-P 4075 4625
-F 0 "#PWR012" H 4075 4375 50  0001 C CNN
-F 1 "GND" H 4080 4452 50  0000 C CNN
-F 2 "" H 4075 4625 50  0001 C CNN
-F 3 "" H 4075 4625 50  0001 C CNN
-	1    4075 4625
-	1    0    0    -1
-$EndComp
-Wire Wire Line
-	4075 4625 4075 4525
-Wire Wire Line
-	4075 3675 4075 3775
-Wire Wire Line
-	4075 4075 4075 4225
+P 4225 4625
+F 0 "#PWR012" H 4225 4375 50  0001 C CNN
+F 1 "GND" H 4230 4452 50  0000 C CNN
+F 2 "" H 4225 4625 50  0001 C CNN
+F 3 "" H 4225 4625 50  0001 C CNN
+	1    4225 4625
+	1    0    0    -1
+$EndComp
+Wire Wire Line
+	4225 4625 4225 4525
+Wire Wire Line
+	4225 3675 4225 3775
+Wire Wire Line
+	4225 4075 4225 4225
 $Comp
 L power:+3.3V #PWR011
 U 1 1 5F8D77CD
-P 4075 3675
-F 0 "#PWR011" H 4075 3525 50  0001 C CNN
-F 1 "+3.3V" H 4090 3848 50  0000 C CNN
-F 2 "" H 4075 3675 50  0001 C CNN
-F 3 "" H 4075 3675 50  0001 C CNN
-	1    4075 3675
+P 4225 3675
+F 0 "#PWR011" H 4225 3525 50  0001 C CNN
+F 1 "+3.3V" H 4240 3848 50  0000 C CNN
+F 2 "" H 4225 3675 50  0001 C CNN
+F 3 "" H 4225 3675 50  0001 C CNN
+	1    4225 3675
 	1    0    0    -1
 $EndComp
@@
 P 2150 4350
 F 0 "D1" H 2150 4133 50  0000 C CNN
-F 1 "1N4148WT" H 2150 4224 50  0000 C CNN
-F 2 "Diode_SMD:D_SOD-523" H 2150 4175 50  0001 C CNN
-F 3 "https://www.diodes.com/assets/Datasheets/ds30396.pdf" H 2150 4350 50  0001 C CNN
+F 1 "SS22T3G" H 2150 4224 50  0000 C CNN
+F 2 "Diode_SMD:D_SMB" H 2150 4175 50  0001 C CNN
+F 3 "https://www.onsemi.com/pdf/datasheet/ss24-d.pdf" H 2150 4350 50  0001 C CNN
 	1    2150 4350
 	-1   0    0    1
@@
 L Device:LED DS3
 U 1 1 60D1DBAD
-P 4675 4375
-F 0 "DS3" V 4713 4258 50  0000 R CNN
-F 1 "LED" V 4622 4258 50  0000 R CNN
-F 2 "LED_SMD:LED_1206_3216Metric_Pad1.42x1.75mm_HandSolder" H 4675 4375 50  0001 C CNN
-F 3 "~" H 4675 4375 50  0001 C CNN
-	1    4675 4375
+P 4850 4375
+F 0 "DS3" V 4888 4258 50  0000 R CNN
+F 1 "LED" V 4797 4258 50  0000 R CNN
+F 2 "LED_SMD:LED_1206_3216Metric_Pad1.42x1.75mm_HandSolder" H 4850 4375 50  0001 C CNN
+F 3 "~" H 4850 4375 50  0001 C CNN
+	1    4850 4375
 	0    -1   -1   0
 $EndComp
@@
 L Device:R R5
 U 1 1 60D1DBB3
-P 4675 3925
-F 0 "R5" H 4745 3971 50  0000 L CNN
-F 1 "820R" H 4745 3880 50  0000 L CNN
-F 2 "Resistor_SMD:R_0805_2012Metric_Pad1.15x1.40mm_HandSolder" V 4605 3925 50  0001 C CNN
-F 3 "~" H 4675 3925 50  0001 C CNN
-	1    4675 3925
+P 4850 3925
+F 0 "R5" H 4920 3971 50  0000 L CNN
+F 1 "820R" H 4920 3880 50  0000 L CNN
+F 2 "Resistor_SMD:R_0805_2012Metric_Pad1.15x1.40mm_HandSolder" V 4780 3925 50  0001 C CNN
+F 3 "~" H 4850 3925 50  0001 C CNN
+	1    4850 3925
 	1    0    0    -1
 $EndComp
@@
 L power:GND #PWR014
 U 1 1 60D1DBB9
-P 4675 4625
-F 0 "#PWR014" H 4675 4375 50  0001 C CNN
-F 1 "GND" H 4680 4452 50  0000 C CNN
-F 2 "" H 4675 4625 50  0001 C CNN
-F 3 "" H 4675 4625 50  0001 C CNN
-	1    4675 4625
-	1    0    0    -1
-$EndComp
-Wire Wire Line
-	4675 4625 4675 4525
-Wire Wire Line
-	4675 4075 4675 4225
-Text Label 4325 3550 0    50   ~ 0
-VAR_VLG
-Wire Wire Line
-	4675 3550 4325 3550
-Wire Wire Line
-	4675 3550 4675 3775
+P 4850 4625
+F 0 "#PWR014" H 4850 4375 50  0001 C CNN
+F 1 "GND" H 4855 4452 50  0000 C CNN
+F 2 "" H 4850 4625 50  0001 C CNN
+F 3 "" H 4850 4625 50  0001 C CNN
+	1    4850 4625
+	1    0    0    -1
+$EndComp
+Wire Wire Line
+	4850 4625 4850 4525
+Wire Wire Line
+	4850 4075 4850 4225
+Text Label 4500 3550 0    50   ~ 0
+VAR_VLG
+Wire Wire Line
+	4850 3550 4500 3550
+Wire Wire Line
+	4850 3550 4850 3775
 $Comp
 L Connector_Generic:Conn_02x04_Odd_Even J6
@@
 Wire Wire Line
 	9475 1850 9875 1850
+Text Notes 3575 4450 1    50   ~ 0
+RED
+Text Notes 4150 4450 1    50   ~ 0
+RED
+Text Notes 4775 4450 1    50   ~ 0
+RED
+Text Notes 2775 6550 0    50   ~ 0
+Use 2k pot\nif available
 $EndSCHEMATC

Commit message: Calculations added
Other:
- note added: "# Reverse voltage protection diode\n\nImax = 2A \nVrev-max = 20V\nVf = 0.3V - 0.4V for ≈1A\n\n--------------------------------------------\n"
- note added: "# Variable voltage supply\n\nVout = 1.25 * (1+ (R2/R1))\n\nVout-max = Vin = 12V\nSubstituting Vout = 12V and R1 = 240 ohm we get R2 ≈ 2 kohm\n--------------------------------------------"
- note added: "--------------------------------------------\n# Current limiting resistor\n\nR = (Vs - Vled)/Iled\nVled-red = 2V typical\n\nR @ 5V = 2.2k Iled = 1.3 mA\nR @ 3.3V = 1.5k Iled = 1.3 mA\nR @ var = 820R Iled =10.9 mA (At Vs-max = 12V)\n--------------------------------------------"
- note added: "AMS-1117 voltage regulators features\n\n- Low dropout voltage\n- Both 5V and 3.3V variant available\n- Maximum current = 1.1 A\n\n"
- note added: "Calculations"
