File: THT/board.kicad_pcb (KiCad board)
At the start: 2 copper layers, 30 x 60 mm, 22 parts, among them J1 9V Battery, J2 USB_B, J3 Barrel_Jack_Switch, J4 1, J5 2, J6 3, SW1 SW_DIP_x03, U1 AMS1117-5.0, U2 AMS1117-3.3

Commit message: THT Kicad 10
Parts:
- removed  5V: TestPoint, TestPoint:TestPoint_Pad_1.0x1.0mm
- removed 3V3: TestPoint, TestPoint:TestPoint_Pad_1.0x1.0mm
- removed Polarity: Symbol_Barrel_Polarity, Symbol:Symbol_Barrel_Polarity
- removed REF**: OSHW-Logo2_7.3x6mm_SilkScreen, Symbol:OSHW-Logo2_7.3x6mm_SilkScreen
- added 3.3V: TestPoint, TestPoint:TestPoint_Pad_1.0x1.0mm, F.Cu at (138.0, 78.0)
- added 5V: TestPoint, TestPoint:TestPoint_Pad_1.0x1.0mm, F.Cu at (135.0, 78.0)
- J2: footprint Breadboard_Power_Supply:USB_B_OST_USB-B1HSxx_Horizontal -> Board:USB_B_OST_USB-B1HSxx_Horizontal
- J3: footprint Breadboard_Power_Supply:BarrelJack_CUI_PJ-102AH_Horizontal -> Board:BarrelJack_CUI_PJ-102AH_Horizontal
- moved VIN 2.65 mm to (135.0, 74.8)
- moved GND 1.70 mm to (138.0, 74.8)
- moved J5 0.18 mm to (159.7, 116.3)
- moved J4 0.13 mm to (159.6, 65.3)
Connections:
- net +3V3 renamed +3.3V
- net 3.3V_OUT renamed /3.3V
- net 5V_OUT renamed /5V
- net VIN renamed /VIN
- J2 pad 2: Net-(J2-Pad2) -> unconnected-(J2-D--Pad2)
- J2 pad 3: Net-(J2-Pad3) -> unconnected-(J2-D+-Pad3)
- J2 pad 4: Net-(J2-Pad4) -> unconnected-(J2-GND-Pad4)
Routing:
- net GND: track 0.00 -> 151.4 mm, vias 0 -> 1
- net /5V: track 22.4 -> 44.2 mm, vias 0 -> 2
- net /VIN: track 31.9 -> 40.9 mm, vias 0 -> 2
- net +5V: track 54.4 -> 61.6 mm
- net VDC: track 53.5 -> 55.2 mm
- net +3.3V: track 66.0 -> 65.4 mm
- net /3.3V: track 40.2 -> 40.5 mm, vias 0 -> 1
Other:
- rule pad_to_mask_clearance: 0.2 -> 0.05
