File: THT/board.kicad_sch (KiCad schematic)
At the start: 20 parts, among them J1 9V Battery, J2 USB_B, J3 Barrel_Jack_Switch, J4 1, J5 2, J6 3, SW1 SW_DIP_x03, U1 AMS1117-5.0, U2 AMS1117-3.3

Commit message: THT Kicad 10
Parts:
- C1, C2: symbol Device:CP_Small -> Device:C_Polarized_Small
- J1: symbol Connector:Conn_01x02_Female -> Connector:Conn_01x02_Socket
- J2: footprint Breadboard_Power_Supply:USB_B_OST_USB-B1HSxx_Horizontal -> Board:USB_B_OST_USB-B1HSxx_Horizontal; symbol Connector:USB_B -> Board:USB_B
- J3: footprint Breadboard_Power_Supply:BarrelJack_CUI_PJ-102AH_Horizontal -> Board:BarrelJack_CUI_PJ-102AH_Horizontal
Connections:
- net +3.3V: now also SW1.4; no longer SW1.5
- net +5V: now also SW1.6
- net GND: now also J2.5 (Shield); no longer J2.SH (Shield)
- net VDC: now also SW1.2; no longer SW1.1
- net VIN: now also SW1.5; no longer SW1.6
- net 3.3V: now reaches SW1.3
- net 3.3V: now also C2.1, U2.2 (VO)
- removed net 3.3V_OUT: C2.1, SW1.2, U2.2 (VO)
- net 5V_OUT renamed 5V
- net 5V: now also SW1.1
Other:
- moved on the sheet: J6, TP1, TP2, TP3, TP4
